File: cutdown-pcb.kicad_sch (KiCad schematic)
At the start: 6 parts, among them J1 Conn_01x06

Commit message: Version 3
Parts:
- added D1: D, Diode_THT:D_DO-35_SOD27_P10.16mm_Horizontal, symbol Device:D
- added J2: Conn_01x02_Pin, Connector_PinHeader_2.54mm:PinHeader_1x02_P2.54mm_Vertical, symbol Connector:Conn_01x02_Pin
- added U5: ~, CustomFootprints:AdafruitMotorDriverBreakout, symbol CustomSymbols:AdafruitDRV8833MotorDriverBreakout
Connections:
- net +5V: now also D1.2 (A)
- net GND: now also A1.21 (D9), U5.7 (GND)
- net RL1: now also A1.25 (D13); no longer A1.16 (DIO1)
- net RL2: now also A1.24 (D12); no longer A1.32 (DIO2)
- net RL3: now also A1.23 (D11); no longer A1.31 (DIO3)
- net RL4: now also A1.22 (D10); no longer A1.30 (DIO5)
- net at A1.10 (A5): now also U1.4 (CS/D3)
- net at A1.6 (A1): now also U5.1 (AIN1)
- net at A1.7 (A2): now also U5.2 (AIN2)
- net at A1.8 (A3): now also U5.3 (SLP)
- net at A1.9 (A4): now also U5.6 (FLT)
- new net: J2.2 (Pin_2), U5.10 (AOUT2)
- new net: D1.1 (K), U5.8 (VM)
- new net: J2.1 (Pin_1), U5.9 (AOUT1)
- no-connect marks 34 -> 35

Commit message: Final SP '25 Flyable PCB and Cutdown board laser files
Parts:
- added D2: LED, LED_THT:LED_D5.0mm, symbol Device:LED
- added R1: R, Resistor_THT:R_Axial_DIN0207_L6.3mm_D2.5mm_P10.16mm_Horizontal, symbol Device:R
Connections:
- net GND: now also A1.20 (D6), D2.1 (K); no longer A1.21 (D9)
- net SPI_CLK: now reaches A1.11 (SCK/D24), U1.7 (CLK)
- net SPI_MISO: now reaches U1.6 (MISO/D0)
- net SPI_MISO: now also A1.13 (MISO/D22); no longer A1.12 (MOSI/D23)
- net SPI_MOSI: now reaches U1.5 (MOSI/CMD)
- net SPI_MOSI: now also A1.12 (MOSI/D23); no longer A1.13 (MISO/D22)
- net LED: now reaches A1.19 (D5)
- net LED: now also R1.1
- new net: D2.2 (A), R1.2
- no-connect marks 35 -> 34
Other:
- note added: "Status Indicator Green LED"
- title: (none) -> Lightning From The Edge of Space Cutdown Payload
